Commit message: feat: implement pure pursuit tracking control and fix slam toolbox parameter injection

File: src/diff_drive_pkg/urdf/diff_drive_gazebo.urdf.xacro (robot description, xacro)
@@ -8,7 +8,11 @@
       </ros>
       <update_rate>30</update_rate>
-      <left_joint>wheel_left_joint</left_joint>
-      <right_joint>wheel_right_joint</right_joint>
+      <num_wheel_pairs>2</num_wheel_pairs>
+      <left_joint>front_left_wheel_joint</left_joint>
+      <left_joint>rear_left_wheel_joint</left_joint>
+      <right_joint>front_right_wheel_joint</right_joint>
+      <right_joint>rear_right_wheel_joint</right_joint>
       <wheel_separation>${wheel_base}</wheel_separation>
+      <wheel_separation>${wheel_base}</wheel_separation> <wheel_diameter>${wheel_radius * 2}</wheel_diameter>
       <wheel_diameter>${wheel_radius * 2}</wheel_diameter>
       <max_wheel_torque>20</max_wheel_torque>
@@ -44,5 +48,6 @@
         <ros>
           <namespace>/</namespace>
-          <remapping>~/out:=scan</remapping> </ros>
+          <remapping>~/out:=scan</remapping>
+        </ros>
         <output_type>sensor_msgs/LaserScan</output_type>
         <frame_name>laser_link</frame_name>

File: src/diff_drive_pkg/urdf/diff_drive_robot.urdf.xacro (robot description, xacro)
@@ -2,9 +2,10 @@
 <robot name="diff_drive_robot" xmlns:xacro="http://www.ros.org/wiki/xacro">
   <xacro:property name="wheel_radius" value="0.05"/>
-  <xacro:property name="wheel_width" value="0.02"/> <xacro:property name="wheel_base" value="0.3"/>
-  <xacro:property name="chassis_length" value="0.2"/>
+  <xacro:property name="wheel_width" value="0.02"/>
+  <xacro:property name="wheel_base" value="0.3"/> <xacro:property name="chassis_length" value="0.2"/>
   <xacro:property name="chassis_width" value="0.15"/>
   <xacro:property name="chassis_height" value="0.05"/>
-  <xacro:property name="wheel_mass" value="0.5"/> <link name="base_link">
+  <xacro:property name="wheel_mass" value="0.5"/>
+  <link name="base_link">
     <visual>
       <geometry>
@@ -14,4 +15,5 @@
         <color rgba="0 0 1 1"/>
       </material>
+      <origin xyz="0 0 0.02" rpy="0 0 0"/>
     </visual>
     <collision>
@@ -19,4 +21,5 @@
         <box size="${chassis_length} ${chassis_width} ${chassis_height}"/>
       </geometry>
+      <origin xyz="0 0 0.02" rpy="0 0 0"/>
     </collision>
     <inertial>
@@ -25,56 +28,39 @@
     </inertial>
   </link>
-  <link name="wheel_left_link">
-    <visual>
-      <geometry>
-        <cylinder radius="${wheel_radius}" length="${wheel_width}"/>
-      </geometry>
-      <origin xyz="0 0 0" rpy="1.570796 0 0"/> </visual>
-    <collision>
-      <geometry>
-        <cylinder radius="${wheel_radius}" length="${wheel_width}"/>
-      </geometry>
-      <origin xyz="0 0 0" rpy="1.570796 0 0"/>
-    </collision>
-    <inertial>
-      <mass value="${wheel_mass}"/>
-      <inertia ixx="0.001" iyy="0.001" izz="0.001" ixy="0" ixz="0" iyz="0"/>
-    </inertial>
-  </link>
-  <joint name="wheel_left_joint" type="continuous">
-    <parent link="base_link"/>
-    <child link="wheel_left_link"/>
-    <origin xyz="0 ${wheel_base/2} 0" rpy="0 0 0"/>
-    <axis xyz="0 1 0"/>
-  </joint>
-  <link name="wheel_right_link">
-    <visual>
-      <geometry>
-        <cylinder radius="${wheel_radius}" length="${wheel_width}"/>
-      </geometry>
-      <origin xyz="0 0 0" rpy="1.570796 0 0"/>
-    </visual>
-    <collision>
-      <geometry>
-        <cylinder radius="${wheel_radius}" length="${wheel_width}"/>
-      </geometry>
-      <origin xyz="0 0 0" rpy="1.570796 0 0"/>
-    </collision>
-    <inertial>
-      <mass value="${wheel_mass}"/>
-      <inertia ixx="0.001" iyy="0.001" izz="0.001" ixy="0" ixz="0" iyz="0"/>
-    </inertial>
-  </link>
-  <joint name="wheel_right_joint" type="continuous">
-    <parent link="base_link"/>
-    <child link="wheel_right_link"/>
-    <origin xyz="0 -${wheel_base/2} 0" rpy="0 0 0"/>
-    <axis xyz="0 1 0"/>
-  </joint>
+  <xacro:macro name="wheel" params="prefix x_offset y_offset">
+    <link name="${prefix}_wheel_link">
+      <visual>
+        <geometry>
+          <cylinder radius="${wheel_radius}" length="${wheel_width}"/>
+        </geometry>
+        <origin xyz="0 0 0" rpy="1.570796 0 0"/>
+      </visual>
+      <collision>
+        <geometry>
+          <cylinder radius="${wheel_radius}" length="${wheel_width}"/>
+        </geometry>
+        <origin xyz="0 0 0" rpy="1.570796 0 0"/>
+      </collision>
+      <inertial>
+        <mass value="${wheel_mass}"/>
+        <inertia ixx="0.001" iyy="0.001" izz="0.001" ixy="0" ixz="0" iyz="0"/>
+      </inertial>
+    </link>
+    <joint name="${prefix}_wheel_joint" type="continuous">
+      <parent link="base_link"/>
+      <child link="${prefix}_wheel_link"/>
+      <origin xyz="${x_offset} ${y_offset} 0" rpy="0 0 0"/>
+      <axis xyz="0 1 0"/>
+    </joint>
+  </xacro:macro>
+  <xacro:wheel prefix="front_left"  x_offset="0.08"  y_offset="${wheel_base/2}"/>
+  <xacro:wheel prefix="front_right" x_offset="0.08"  y_offset="-${wheel_base/2}"/>
+  <xacro:wheel prefix="rear_left"   x_offset="-0.08" y_offset="${wheel_base/2}"/>
+  <xacro:wheel prefix="rear_right"  x_offset="-0.08" y_offset="-${wheel_base/2}"/>
   <link name="laser_link"/>
   <joint name="laser_joint" type="fixed">
     <parent link="base_link"/>
     <child link="laser_link"/>
-    <origin xyz="0 0 0.05" rpy="0 0 0"/>
+    <origin xyz="0 0 0.12" rpy="0 0 0"/>
   </joint>
 </robot>

Commit message: Improve ROS simulation bringup

File: src/diff_drive_pkg/urdf/diff_drive_gazebo.urdf.xacro (robot description, xacro)
@@ -1,5 +1,28 @@
 <?xml version="1.0"?>
 <robot name="diff_drive_robot_sim" xmlns:xacro="http://www.ros.org/wiki/xacro">
-  <xacro:include filename="$(find diff_drive_pkg)/urdf/diff_drive_robot.urdf.xacro" />
+  <xacro:include filename="$(find diff_drive_pkg)/urdf/diff_drive_robot.urdf.xacro"/>
+  <gazebo reference="base_link">
+    <material>Gazebo/Blue</material>
+  </gazebo>
+  <gazebo reference="front_left_wheel_link">
+    <material>Gazebo/Black</material>
+    <mu1>1.0</mu1>
+    <mu2>1.0</mu2>
+  </gazebo>
+  <gazebo reference="front_right_wheel_link">
+    <material>Gazebo/Black</material>
+    <mu1>1.0</mu1>
+    <mu2>1.0</mu2>
+  </gazebo>
+  <gazebo reference="rear_left_wheel_link">
+    <material>Gazebo/Black</material>
+    <mu1>1.0</mu1>
+    <mu2>1.0</mu2>
+  </gazebo>
+  <gazebo reference="rear_right_wheel_link">
+    <material>Gazebo/Black</material>
+    <mu1>1.0</mu1>
+    <mu2>1.0</mu2>
+  </gazebo>
   <gazebo>
     <plugin name="diff_drive" filename="libgazebo_ros_diff_drive.so">
@@ -7,5 +30,5 @@
         <namespace>/</namespace>
       </ros>
-      <update_rate>30</update_rate>
+      <update_rate>50</update_rate>
       <num_wheel_pairs>2</num_wheel_pairs>
       <left_joint>front_left_wheel_joint</left_joint>
@@ -14,8 +37,9 @@
       <right_joint>rear_right_wheel_joint</right_joint>
       <wheel_separation>${wheel_base}</wheel_separation>
-      <wheel_separation>${wheel_base}</wheel_separation> <wheel_diameter>${wheel_radius * 2}</wheel_diameter>
       <wheel_diameter>${wheel_radius * 2}</wheel_diameter>
       <max_wheel_torque>20</max_wheel_torque>
-      <max_wheel_acceleration>1.0</max_wheel_acceleration>
+      <max_wheel_acceleration>2.0</max_wheel_acceleration>
+      <command_topic>cmd_vel</command_topic>
+      <odometry_topic>odom</odometry_topic>
       <publish_odom>true</publish_odom>
       <publish_odom_tf>true</publish_odom_tf>
@@ -33,5 +57,5 @@
         <scan>
           <horizontal>
-            <samples>360</samples>
+            <samples>720</samples>
             <resolution>1</resolution>
             <min_angle>-3.14159</min_angle>
@@ -40,8 +64,13 @@
         </scan>
         <range>
-          <min>0.15</min>
-          <max>10.0</max>
+          <min>0.12</min>
+          <max>8.0</max>
           <resolution>0.01</resolution>
         </range>
+        <noise>
+          <type>gaussian</type>
+          <mean>0.0</mean>
+          <stddev>0.01</stddev>
+        </noise>
       </ray>
       <plugin name="laser_controller" filename="libgazebo_ros_ray_sensor.so">
