Commit message: Clean RViz robot and SLAM warnings

File: src/diff_drive_pkg/urdf/diff_drive_robot.urdf.xacro (robot description, xacro)
@@ -7,4 +7,10 @@
   <xacro:property name="chassis_height" value="0.05"/>
   <xacro:property name="wheel_mass" value="0.5"/>
+  <link name="base_footprint"/>
+  <joint name="base_footprint_joint" type="fixed">
+    <parent link="base_footprint"/>
+    <child link="base_link"/>
+    <origin xyz="0 0 0" rpy="0 0 0"/>
+  </joint>
   <link name="base_link">
     <visual>
